File: Hardware/Nível Digital/nivel_digital.brd (EAGLE design)
At the start: 68.6 x 53.3 mm, 9 parts

Commit message: Botão range adicionado
Parts:
- added S4: (no value), GEAP:B3F-10XX
- moved S2 8.39 mm to (7.37, 11.9)
- moved S3 8.13 mm to (15.5, 12.2)
- moved S1 7.64 mm to (32.8, 12.5)
Connections:
- removed net VCC: U$2.VCC
- new net HOLD: S3.1, S3.2
- new net N$1: U$1.SCL
- new net N$2: U$1.SDA
- new net RANGE: S4.1, S4.2
- new net ZERO: S2.1, S2.2
- net +3V3: now also U$2.VCC
- net +5V: now also U$1.VCC
- net GND: now also S2.3, S2.4, S3.3, S3.4, S4.3, S4.4, U$1.GND
Changed lines of the file:
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@@
 <layer number="17" name="Pads" color="2" fill="1" visible="yes" active="yes"/>
 <layer number="18" name="Vias" color="14" fill="1" visible="yes" active="yes"/>
-<layer number="19" name="Unrouted" color="11" fill="1" visible="yes" active="yes"/>
+<layer number="19" name="Unrouted" color="16" fill="1" visible="yes" active="yes"/>
 <layer number="20" name="Dimension" color="15" fill="1" visible="yes" active="yes"/>
 <layer number="21" name="tPlace" color="7" fill="1" visible="yes" active="yes"/>
@@
 <attribute name="VALUE" x="32.512" y="-1.778" locked="yes" size="1.27" layer="27"/>
 </element>
-<element name="S1" library="GEAP" package="B3F-10XX" package3d_urn="urn:adsk.eagle:package:35685920/2" value="" x="25.146" y="12.0396" smashed="yes" rot="R270">
-<attribute name="NAME" x="28.829" y="15.0876" size="1.27" layer="25" ratio="10" rot="R270"/>
-<attribute name="VALUE" x="20.066" y="15.0876" size="1.27" layer="27" ratio="10" rot="R270"/>
+<element name="S1" library="GEAP" package="B3F-10XX" package3d_urn="urn:adsk.eagle:package:35685920/2" value="" x="32.766" y="12.5476" smashed="yes" rot="R270">
+<attribute name="NAME" x="36.449" y="15.5956" size="1.27" layer="25" ratio="10" rot="R270"/>
+<attribute name="VALUE" x="27.686" y="15.5956" size="1.27" layer="27" ratio="10" rot="R270"/>
 </element>
 <element name="U$1" library="GEAP" package="OLED_0.96_I2C" package3d_urn="urn:adsk.eagle:package:30876132/2" value="" x="16.764" y="33.528" smashed="yes"/>
 <element name="U$2" library="GEAP" package="MODULO_ADXL345" override_package3d_urn="urn:adsk.eagle:package:35821945/2" override_package_urn="urn:adsk.eagle:footprint:35821946/1" value="MODULO_ADXL345" x="34.798" y="17.272" smashed="yes"/>
-<element name="S2" library="GEAP" package="B3F-10XX" package3d_urn="urn:adsk.eagle:package:35685920/2" value="" x="15.748" y="12.192" smashed="yes" rot="R90">
-<attribute name="NAME" x="12.065" y="9.144" size="1.27" layer="25" ratio="10" rot="R90"/>
-<attribute name="VALUE" x="20.828" y="9.144" size="1.27" layer="27" ratio="10" rot="R90"/>
-</element>
-<element name="S3" library="GEAP" package="B3F-10XX" package3d_urn="urn:adsk.eagle:package:35685920/2" value="" x="7.366" y="12.192" smashed="yes" rot="R90">
-<attribute name="NAME" x="3.683" y="9.144" size="1.27" layer="25" ratio="10" rot="R90"/>
-<attribute name="VALUE" x="12.446" y="9.144" size="1.27" layer="27" ratio="10" rot="R90"/>
+<element name="S2" library="GEAP" package="B3F-10XX" package3d_urn="urn:adsk.eagle:package:35685920/2" value="" x="7.366" y="11.938" smashed="yes" rot="R90">
+<attribute name="NAME" x="3.683" y="8.89" size="1.27" layer="25" ratio="10" rot="R90"/>
+<attribute name="VALUE" x="12.446" y="8.89" size="1.27" layer="27" ratio="10" rot="R90"/>
+</element>
+<element name="S3" library="GEAP" package="B3F-10XX" package3d_urn="urn:adsk.eagle:package:35685920/2" value="" x="15.494" y="12.192" smashed="yes" rot="R90">
+<attribute name="NAME" x="11.811" y="9.144" size="1.27" layer="25" ratio="10" rot="R90"/>
+<attribute name="VALUE" x="20.574" y="9.144" size="1.27" layer="27" ratio="10" rot="R90"/>
+</element>
+<element name="S4" library="GEAP" package="B3F-10XX" package3d_urn="urn:adsk.eagle:package:35685920/2" value="" x="23.114" y="12.192" smashed="yes" rot="R90">
+<attribute name="NAME" x="19.431" y="9.144" size="1.27" layer="25" ratio="10" rot="R90"/>
+<attribute name="VALUE" x="28.194" y="9.144" size="1.27" layer="27" ratio="10" rot="R90"/>
 </element>
 </elements>
@@
 <contactref element="POWER" pad="5"/>
 <contactref element="POWER" pad="2"/>
-<wire x1="30.48" y1="2.54" x2="38.1" y2="2.54" width="0" layer="19" extent="1-1"/>
+<contactref element="U$1" pad="VCC"/>
+<wire x1="30.48" y1="2.54" x2="12.594" y2="45.158" width="0" layer="19" extent="1-1"/>
+<wire x1="38.1" y1="2.54" x2="30.48" y2="2.54" width="0" layer="19" extent="1-1"/>
 </signal>
 <signal name="GND" class="2">
@@
 <contactref element="S1" pad="3"/>
 <contactref element="U$2" pad="GND"/>
+<contactref element="S4" pad="4"/>
+<contactref element="S2" pad="3"/>
+<contactref element="S2" pad="4"/>
+<contactref element="S3" pad="3"/>
+<contactref element="S3" pad="4"/>
+<contactref element="S4" pad="3"/>
+<contactref element="U$1" pad="GND"/>
+<wire x1="15.134" y1="45.158" x2="26.416" y2="50.8" width="0" layer="19" extent="1-1"/>
 <wire x1="36.068" y1="36.322" x2="26.416" y2="50.8" width="0" layer="19" extent="1-1"/>
-<wire x1="22.8854" y1="15.2908" x2="36.068" y2="36.322" width="0" layer="19" extent="1-1"/>
-<wire x1="22.8854" y1="8.7884" x2="22.8854" y2="15.2908" width="0" layer="19" extent="1-1"/>
-<wire x1="40.64" y1="2.54" x2="22.8854" y2="8.7884" width="0" layer="19" extent="1-1"/>
+<wire x1="30.5054" y1="15.7988" x2="36.068" y2="36.322" width="0" layer="19" extent="1-1"/>
+<wire x1="9.6266" y1="15.1892" x2="30.5054" y2="15.7988" width="0" layer="19" extent="1-1"/>
+<wire x1="30.5054" y1="9.2964" x2="30.5054" y2="15.7988" width="0" layer="19" extent="1-1"/>
+<wire x1="9.6266" y1="8.6868" x2="30.5054" y2="9.2964" width="0" layer="19" extent="1-1"/>
+<wire x1="17.7546" y1="15.4432" x2="9.6266" y2="15.1892" width="0" layer="19" extent="1-1"/>
+<wire x1="17.7546" y1="8.9408" x2="17.7546" y2="15.4432" width="0" layer="19" extent="1-1"/>
+<wire x1="25.3746" y1="15.4432" x2="17.7546" y2="8.9408" width="0" layer="19" extent="1-1"/>
+<wire x1="25.3746" y1="8.9408" x2="25.3746" y2="15.4432" width="0" layer="19" extent="1-1"/>
+<wire x1="40.64" y1="2.54" x2="30.5054" y2="9.2964" width="0" layer="19" extent="1-1"/>
 <wire x1="43.18" y1="2.54" x2="40.64" y2="2.54" width="0" layer="19" extent="1-1"/>
 </signal>
@@
 <signal name="+3V3">
 <contactref element="POWER" pad="4"/>
+<contactref element="U$2" pad="VCC"/>
+<wire x1="35.56" y1="2.54" x2="36.068" y2="33.782" width="0" layer="19" extent="1-1"/>
 </signal>
 <signal name="MISO">
@@
 <contactref element="S1" pad="2"/>
 <contactref element="S1" pad="1"/>
-<wire x1="27.4066" y1="8.7884" x2="27.4066" y2="15.2908" width="0" layer="19" extent="1-1"/>
-<wire x1="33.02" y1="2.54" x2="27.4066" y2="8.7884" width="0" layer="19" extent="1-1"/>
+<wire x1="35.0266" y1="9.2964" x2="35.0266" y2="15.7988" width="0" layer="19" extent="1-1"/>
+<wire x1="33.02" y1="2.54" x2="35.0266" y2="9.2964" width="0" layer="19" extent="1-1"/>
 </signal>
 <signal name="SCK">
 <contactref element="IOH" pad="6"/>
 </signal>
-<signal name="VCC">
-<contactref element="U$2" pad="VCC"/>
+<signal name="ZERO">
+<contactref element="S2" pad="1"/>
+<contactref element="S2" pad="2"/>
+<wire x1="5.1054" y1="8.6868" x2="5.1054" y2="15.1892" width="0" layer="19" extent="1-1"/>
+</signal>
+<signal name="HOLD">
+<contactref element="S3" pad="1"/>
+<contactref element="S3" pad="2"/>
+<wire x1="13.2334" y1="8.9408" x2="13.2334" y2="15.4432" width="0" layer="19" extent="1-1"/>
+</signal>
+<signal name="RANGE">
+<contactref element="S4" pad="1"/>
+<contactref element="S4" pad="2"/>
+<wire x1="20.8534" y1="8.9408" x2="20.8534" y2="15.4432" width="0" layer="19" extent="1-1"/>
+</signal>
+<signal name="N$1">
+<contactref element="U$1" pad="SCL"/>
+</signal>
+<signal name="N$2">
+<contactref element="U$1" pad="SDA"/>
 </signal>
 </signals>
